Commit message: Adding xacro robot model

File: description/robot_core.xacro (robot description, xacro)
@@ -1,4 +1,5 @@
 <?xml version="1.0"?>
 <robot xmlns:xacro="http://www.ros.org/wiki/xacro" >
+    <xacro:include filename="inertial_macros.xacro" />
 <material name="white">
     <color rgba="1 1 1 1" />
@@ -30,4 +31,13 @@
         <material name="white" />
     </visual>
+    <collision>
+        <origin xyz="0.15 0 0.075"/>
+        <geometry>
+            <box size="0.3 0.3 0.15" />
+        </geometry>
+    </collision>
+    <xacro:inertial_box mass="0.5" x="0.3" y ="0.3" z="0.15">
+        <origin xyz="0.15 0 0.075" rpy="0 0 0"/>
+    </xacro:inertial_box>
 </link>
 <!-- LEFT WHEEL LINK-->
@@ -45,4 +55,12 @@
         <material name="blue"/>
     </visual>
+    <collision>
+        <geometry>
+            <cylinder radius="0.05" length="0.04" />
+        </geometry>
+    </collision>
+    <xacro:inertial_cylinder mass="0.1" length="0.04" radius ="0.05">
+        <origin xyz="0 0 0" rpy="0 0 0"/>
+    </xacro:inertial_cylinder>
 </link>
 <!-- RIGHT WHEEL LINK-->
@@ -60,4 +78,12 @@
         <material name="blue"/>
     </visual>
+        <collision>
+        <geometry>
+            <cylinder radius="0.05" length="0.04" />
+        </geometry>
+        </collision>
+    <xacro:inertial_cylinder mass="0.1" length="0.04" radius ="0.05">
+        <origin xyz="0 0 0" rpy="0 0 0"/>
+    </xacro:inertial_cylinder>
 </link>
 <!-- CASTER WHEEL LINK -->
@@ -74,4 +100,12 @@
     <material name="black"/>
 </visual>
+<collision>
+    <geometry>
+        <sphere radius="0.05"/>
+    </geometry>
+</collision>
+    <xacro:inertial_sphere mass="0.1" radius ="0.05">
+        <origin xyz="0 0 0" rpy="0 0 0"/>
+    </xacro:inertial_sphere>
 </link>
 </robot>
