Commit message: qorking getting bounce to stop

File: description/gazebo_control.xacro (robot description, xacro)
@@ -5,12 +5,19 @@
       filename="gz-sim-diff-drive-system"
       name="gz::sim::systems::DiffDrive">
+      <!-- Wheel Information -->
     <left_joint>left_wheel_joint</left_joint>
     <right_joint>right_wheel_joint</right_joint>
+    <!-- Robot geometry -->
     <wheel_separation>0.35</wheel_separation>
     <wheel_radius>0.05</wheel_radius>
+    <!-- ROS topic -->
     <topic>cmd_vel</topic>
+    <!-- Odometry -->
     <odom_topic>odom</odom_topic>
     <frame_id>odom</frame_id>
     <child_frame_id>base_link</child_frame_id>
+    <!-- Optional -->
+     <publish_odom>true</publish_odom>
+     <publish_tf>true</publish_tf>
   </plugin>
 </gazebo>

File: description/robot_core.xacro (robot description, xacro)
@@ -96,5 +96,5 @@
 <visual>
     <geometry>
-        <sphere radius="0.05"/>
+        <sphere radius="0.048"/>
     </geometry>
     <material name="black"/>
@@ -102,8 +102,24 @@
 <collision>
     <geometry>
-        <sphere radius="0.05"/>
+        <sphere radius="0.048"/>
     </geometry>
+  <surface>
+    <friction>
+      <ode>
+        <mu>0.0</mu>
+        <mu2>0.0</mu2>
+      </ode>
+    </friction>
+    <contact>
+      <ode>
+        <kp>100000</kp>
+        <kd>100</kd>
+        <max_vel>0.01</max_vel>
+        <min_depth>0.001</min_depth>
+      </ode>
+    </contact>
+  </surface>
 </collision>
-    <xacro:inertial_sphere mass="0.1" radius ="0.05">
+    <xacro:inertial_sphere mass="0.1" radius="0.048">
         <origin xyz="0 0 0" rpy="0 0 0"/>
     </xacro:inertial_sphere>
